File: GamingController/GamingController.kicad_sch (KiCad schematic)
At the start: 7 parts, among them J1 USB_C_Receptacle_USB2.0_16P, U1 STM32F401RETx, U2 LD3985M33R_SOT23

Commit message: Added Some
Parts:
- added C10: 1uC, symbol Device:C
- added C11, C12, C6, C7, C8, C9: 100nF, symbol Device:C
- added C13, C4: 100n, symbol Device:C
- added C3: 10n, symbol Device:C
- added C5: 1u, symbol Device:C
- added R3: 100k, symbol Device:R
- added R4, R5: 0R, symbol Device:R
- added Y1: ECS-2520MV-xxx-xx, Oscillator:Oscillator_SMD_ECS_2520MV-xxx-xx-4Pin_2.5x2.0mm, symbol Oscillator:ECS-2520MV-xxx-xx
- C2: value 100n -> 1u
Connections:
- net GND is gone; now on net +3V3: J1.A1 (GND), J1.A12 (GND), J1.B1 (GND), J1.B12 (GND), J1.S1 (SHIELD), R1.1, R2.1
- net at C1.1: now also J1.A4 (VBUS), J1.A9 (VBUS), J1.B4 (VBUS), J1.B9 (VBUS), U2.1 (VIN), U2.3 (INH), C5.1
- net +3V3: now reaches C1.2
- net +3V3: now also C2.1, C2.2, U1.1 (VBAT), U1.12 (VSSA), U1.13 (VREF+), U1.18 (VSS), U1.19 (VDD), U1.31 (VSS), U1.32 (VDD), U1.47 (VSS), U1.48 (VDD), U1.60 (BOOT0), U1.63 (VSS), U1.64 (VDD), U2.2 (GND), U2.4 (BYP), C10.2, C11.1, C11.2, C12.2, C13.1, C13.2, C3.1, C3.2, C4.1, C4.2, C5.2, C6.1, C6.2, C7.1, C7.2, C8.1, C8.2, C9.1, C9.2, R3.2, R5.1, R5.2, Y1.1 (Tri-State), Y1.2 (GND), Y1.4 (VDD)
- net at U1.30 (VCAP1): now also C10.1
- net OSC: now reaches U1.5 (PH0)
- net OSC: now also R4.1
- net at U1.7 (NRST): now also C12.1, R3.1
- new net: R4.2, Y1.3 (OUT)
Other:
- moved on the sheet: C1, C2, R1, R2, U2

Commit message: update
Parts:
- removed C12: 100nF, symbol Device:C
- removed R3: 100k, symbol Device:R
- added C11: 100nF, symbol Device:C
- added J2: Conn_01x05, symbol Connector_Generic:Conn_01x05
- added SW1: SW_MEC_5G, symbol Switch:SW_MEC_5G
- added U2: TVS0500DRV, Package_SON:WSON-6-1EP_2x2mm_P0.65mm_EP1x1.6mm, symbol Power_Protection:TVS0500DRV
- added U3: USBLC6-2P6, Package_TO_SOT_SMD:SOT-666, symbol Power_Protection:USBLC6-2P6
- C9: renamed from C6; value 100nF -> 1uF
- renumbered C5 to C1, C11 to C10, C13 to C12, C10 to C13, C1 to C2, C2 to C4, C4 to C5, C9 to C6, C8 to C7, C7 to C8, R5 to R3, U2 to U1, U1 to U4
Connections:
- net +3V3: now also C11.2, J2.1 (Pin_1), J2.5 (Pin_5), SW1.3 (B), SW1.4 (B), U2.1 (GND), U2.2 (GND), U2.3 (GND), U2.7 (GND), U3.2 (GND)
- net NRST: now reaches U4.7 (NRST)
- net NRST: now also C11.1, J2.2 (Pin_2), SW1.1 (A), SW1.2 (A)
- net 5V_VBUS: now reaches C1.1, C2.1, J1.A4 (VBUS), J1.A9 (VBUS), J1.B4 (VBUS), J1.B9 (VBUS), U1.1 (VIN), U1.3 (INH)
- net 5V_VBUS: now also U2.4 (IN), U2.5 (IN), U2.6 (IN), U3.5 (VBUS)
- net at J1.A6 (D+): now also J1.B6 (D+), U3.3 (I/O2)
- net at J1.A7 (D-): now also J1.B7 (D-), U3.1 (I/O1)
- net Thumb_R.X: now reaches U4.20 (PA4)
- net Thumb_R.Y: now reaches U4.21 (PA5)
- net Thumb_L.X: now reaches U4.22 (PA6)
- net Thumb_L.Y: now reaches U4.23 (PA7)
- net USB.D N: now reaches U4.44 (PA11)
- net USB.D N: now also U3.6 (I/O1)
- net USB.D P: now reaches U4.45 (PA12)
- net USB.D P: now also U3.4 (I/O2)
- net SWD.SWDIO: now reaches U4.46 (PA13)
- net SWD.SWDIO: now also J2.3 (Pin_3)
- net SWD.SWCLK: now reaches U4.49 (PA14)
- net SWD.SWCLK: now also J2.4 (Pin_4)
- no-connect marks 0 -> 2
Other:
- added sheet User Interface (user_interface.kicad_sch)
- note added: "Oscillator"
- note added: "Protection Circuit"
- note added: "Reset Btn"
- note added: "SWD Receiver"
- note added: "Voltage Regulator"
- title: (none) -> STM32_GamingController
- moved on the sheet: C1, C2, C3, C4, C5, J1, R1, R2, U1

Commit message: forgot to save
Changed lines of the file:
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@@
 	)
 	(sheet
-		(at 210.185 125.095)
-		(size 32.385 21.59)
+		(at 197.485 102.87)
+		(size 59.69 38.735)
 		(exclude_from_sim no)
 		(in_bom yes)
@@
 		)
 		(property "Sheetname" "User Interface"
-			(at 210.185 124.3834 0)
+			(at 197.485 102.1584 0)
 			(effects
 				(font
@@
 		)
 		(property "Sheetfile" "user_interface.kicad_sch"
-			(at 210.185 147.2696 0)
+			(at 197.485 142.1896 0)
 			(effects
 				(font

Commit message: Draw Schematics
Parts:
- removed J2: Conn_01x05, symbol Connector_Generic:Conn_01x05
- removed R3, R4: 0R, symbol Device:R
- removed SW1: SW_MEC_5G, symbol Switch:SW_MEC_5G
- added C14: 4.7u, Capacitor_SMD:C_0201_0603Metric, symbol Device:C_Small
- added IC1: BMD-330-A-R, BD330:BMD330AR, symbol BMD-330-A-R:BMD-330-A-R
- added J2, J3: Conn_01x05_Socket, Connector_PinSocket_2.00mm:PinSocket_1x05_P2.00mm_Horizontal, symbol Connector:Conn_01x05_Socket
- added S14: DTS-63N-V, TactSwitch:DTS63NV, symbol DTS-63N-V:DTS-63N-V
- C1, C4: value 1u -> 1u_X5R_0603; footprint (none) -> Capacitor_SMD:C_0201_0603Metric
- C10, C11, C12, C13, C2, C5, C6, C7, C8, C9: footprint (none) -> Capacitor_SMD:C_0201_0603Metric
- C3: value 10n -> 10nF_X7R_0603; footprint (none) -> Capacitor_SMD:C_0201_0603Metric
- J1: footprint (none) -> Connector_USB:USB_C_Receptacle_JAE_DX07S016JA1R1500
- R1, R2: footprint (none) -> Resistor_SMD:R_0201_0603Metric
- renumbered U3 to U1, U1 to U3
Connections:
- net +3V3: now also U3.5 (VOUT), C14.1, IC1.17 (VCC), J2.1 (Pin_1), J3.1 (Pin_1); no longer C1.2, C10.2, C11.2, C12.2, C13.2, C2.2, C3.1, C3.2, C4.2, C5.2, C6.2, C7.2, C8.2, C9.2, J1.A1 (GND), J1.A12 (GND), J1.B1 (GND), J1.B12 (GND), J1.S1 (SHIELD), R1.1, R2.1, U1.2 (GND), U2.1 (GND), U2.2 (GND), U2.3 (GND), U2.7 (GND), U3.2 (GND), U3.4 (BYP), U4.1 (VBAT), U4.12 (VSSA), U4.18 (VSS), U4.31 (VSS), U4.47 (VSS), U4.60 (BOOT0), U4.63 (VSS), Y1.2 (GND)
- net NRST: now also J2.2 (Pin_2), S14.1 (COM_1)
- net OSC: now also Y1.3 (OUT)
- net SWD.SWCLK: now also J2.4 (Pin_4)
- net SWD.SWDIO: now also J2.3 (Pin_3)
- net Thumb_L.X: now also U4.11 (PC3); no longer U4.22 (PA6)
- net Thumb_L.Y: now also U4.24 (PC4); no longer U4.23 (PA7)
- net Thumb_R.X: now also U4.9 (PC1); no longer U4.20 (PA4)
- net Thumb_R.Y: now also U4.10 (PC2); no longer U4.21 (PA5)
- net DPAD.S: now reaches U4.2 (PC13)
- net BTN.PS: now reaches U4.25 (PC5)
- net TPad.DR: now reaches U4.26 (PB0)
- net DPAD.W: now reaches U4.3 (PC14)
- net TPad.SS: now reaches U4.33 (PB12)
- net TPad.BTN1: now reaches U4.34 (PB13)
- net TPad.BTN2: now reaches U4.35 (PB14)
- net TPad.BTN3: now reaches U4.36 (PB15)
- net BTN.L1: now reaches U4.37 (PC6)
- net BTN.R1: now reaches U4.38 (PC7)
- net BTN.A: now reaches U4.39 (PC8)
- net DPAD.E: now reaches U4.4 (PC15)
- net BTN.B: now reaches U4.40 (PC9)
- net BTN.X: now reaches U4.51 (PC10)
- net BTN.Y: now reaches U4.52 (PC11)
- net DPAD.N: now reaches U4.53 (PC12)
- net TPad.SCK: now reaches U4.55 (PB3)
- net TPad.MISO: now reaches U4.56 (PB4)
- net TPad.MOSI: now reaches U4.57 (PB5)
- net LCD.SCL: now reaches U4.58 (PB6)
- net LCD.SDA: now reaches U4.59 (PB7)
- net USB.D N renamed USB.D_N
- net USB.D P renamed USB.D_P
- new net: C3.1, U3.4 (BYP)
- new net BLE_SWD.NRST: IC1.39 (P0.21), J3.2 (Pin_2)
- new net BLE_SWD.SWCLK: IC1.43 (SWCLK), J3.4 (Pin_4)
- new net BLE_SWD.SWDIO: IC1.44 (SWDIO), J3.3 (Pin_3)
- new net GND: C1.2, C10.2, C11.2, C12.2, C13.2, C14.2, C2.2, C3.2, C4.2, C5.2, C6.2, C7.2, C8.2, C9.2, IC1.1 (GND_1), IC1.18 (GND_7), IC1.2 (GND_2), IC1.29 (GND_8), IC1.3 (GND_3), IC1.30 (GND_9), IC1.4 (GND_4), IC1.45 (GND_10), IC1.46 (GND_11), IC1.47 (GND_12), IC1.5 (GND_5), J1.A1 (GND), J1.A12 (GND), J1.B1 (GND), J1.B12 (GND), J1.S1 (SHIELD), J2.5 (Pin_5), J3.5 (Pin_5), R1.1, R2.1, S14.3 (NO_1), U1.2 (GND), U2.1 (GND), U2.2 (GND), U2.3 (GND), U2.7 (GND), U3.2 (GND), U4.1 (VBAT), U4.12 (VSSA), U4.18 (VSS), U4.31 (VSS), U4.47 (VSS), U4.60 (BOOT0), U4.63 (VSS), Y1.2 (GND)
- no-connect marks 2 -> 56
Other:
- sheet User Interface ports: added BTN.A, BTN.B, BTN.L1, BTN.PS, BTN.R1, BTN.X, BTN.Y, DPAD.E, DPAD.N, DPAD.S, DPAD.W, LCD.SCL, LCD.SDA, TPad.BTN1, TPad.BTN2, TPad.BTN3, TPad.DR, TPad.MISO, TPad.MOSI, TPad.SCK, TPad.SS, Thumb_L.X, Thumb_L.Y, Thumb_R.X, Thumb_R.Y, Thumb_SW_L, Thumb_SW_R; removed none
- note added: "(BLE)SWD Receiver"
- note added: "Bluetooth Module"
- note added: "Microcontroller"
- moved on the sheet: C10, C11, C12, C4, C6, C7, C8, C9, Y1

Commit message: Schematics Done
Parts:
- added D1: LED, LED_SMD:LED_0201_0603Metric, symbol Device:LED
- added R3: 2k, Resistor_SMD:R_0201_0603Metric, symbol Device:R_Small
Connections:
- net +3V3: now also R3.1
- net GND: now also D1.1 (K)
- net RGB_A.Blue: now reaches U4.14 (PA0)
- net RGB_A.Green: now reaches U4.15 (PA1)
- net RGB_A.Red: now reaches U4.16 (PA2)
- net RGB_B.Blue: now reaches U4.17 (PA3)
- net RGB_B.Green: now reaches U4.20 (PA4)
- net RGB_B.Red: now reaches U4.21 (PA5)
- new net: D1.2 (A), R3.2
- no-connect marks 56 -> 50
Other:
- sheet User Interface ports: added RGB_A.Blue, RGB_A.Green, RGB_A.Red, RGB_B.Blue, RGB_B.Green, RGB_B.Red; removed none
