File: GamingController/user_interface.kicad_sch (KiCad schematic)
At the start: 4 parts

Commit message: forgot to save
Parts:
- removed R5, R6: 10k, symbol Device:R
- added C14, C15, C16, C17, C18, C19, C20, C21, C22, C23, C24, C25, C26, C27, C28: 100n, symbol Device:C_Small
- added R10, R11, R12, R13, R14, R15, R16, R17, R6, R8, R9: 56k, symbol Device:R_Small
- added R5, R7: 10k, symbol Device:R_Small
- added SW10, SW11, SW12, SW2, SW3, SW4, SW5, SW6, SW7, SW8, SW9: SW_Push, Button_Switch_SMD:SW_SPST_Omron_B3FS-101xP, symbol Switch:SW_Push
Connections:
- net +3V3: now also R5.1, R7.1, SW10.1, SW11.1, SW12.1, SW2.1, SW3.1, SW4.1, SW5.1, SW6.1, SW7.1, SW8.1, SW9.1
- net GND: now also C14.2, C15.2, C16.2, C17.2, C18.2, C19.2, C20.2, C21.2, C22.2, C23.2, C24.2, C25.2, C26.2, C27.2, C28.2
- net Thumb_L.X: now also C18.1
- net Thumb_L.Y: now also C17.1
- net Thumb_R.X: now also C16.1
- net Thumb_R.Y: now also C15.1
- net Thumb_SW_L: now also R7.2
- net Thumb_SW_R: now also R5.2
- new net: C27.1, R16.2
- new net: C24.1, R13.2
- new net: C26.1, R15.2
- new net: C14.1, R6.2
- new net: C22.1, R11.2
- new net: C25.1, R14.2
- new net: C21.1, R10.2
- new net: C19.1, R8.2
- new net: C28.1, R17.2
- new net: C23.1, R12.2
- new net: C20.1, R9.2
- new net BTN.A: R6.1, SW2.2
- new net BTN.B: R8.1, SW3.2
- new net BTN.L1: R16.1, SW11.2
- new net BTN.PS: R15.1, SW10.2
- new net BTN.R1: R17.1, SW12.2
- new net BTN.X: R9.1, SW4.2
- new net BTN.Y: R10.1, SW5.2
- new net DPAD.E: R14.1, SW9.2
- new net DPAD.N: R11.1, SW6.2
- new net DPAD.S: R12.1, SW7.2
- new net DPAD.W: R13.1, SW8.2
Other:
- note added: "Buttons"
- note added: "DPADs"
- note added: "UtilBtns"
- moved on the sheet: S2, S3

Commit message: Draw Schematics
Parts:
- removed SW10, SW11, SW12, SW2, SW3, SW4, SW5, SW6, SW7, SW8, SW9: SW_Push, Button_Switch_SMD:SW_SPST_Omron_B3FS-101xP, symbol Switch:SW_Push
- added C30, C31, C32: 1u, Capacitor_SMD:C_0201_0603Metric, symbol Device:C_Small
- added J4: FFC ADAPTER, FFCAdapter:0781271220, symbol 0781271220:0781271220
- added J5: Conn_01x09_Socket, Connector_PinSocket_1.27mm:PinSocket_1x09_P1.27mm_Vertical, symbol Connector:Conn_01x09_Socket
- added R18: 10k, Resistor_SMD:R_0201_0603Metric_Pad0.64x0.40mm_HandSolder, symbol Device:R_Small
- added S10, S11, S12, S13, S3, S4, S5, S6, S7, S8, S9: DTS-63N-V, TactSwitch:DTS63NV, symbol DTS-63N-V:DTS-63N-V
- C15, C16, C17, C18: footprint (none) -> Capacitor_SMD:C_0201_0603Metric
- C19: renamed from C14; footprint (none) -> Capacitor_SMD:C_0201_0603Metric
- C20: renamed from C19; footprint (none) -> Capacitor_SMD:C_0201_0603Metric
- C21: renamed from C20; footprint (none) -> Capacitor_SMD:C_0201_0603Metric
- C22: renamed from C21; footprint (none) -> Capacitor_SMD:C_0201_0603Metric
- C23: renamed from C22; footprint (none) -> Capacitor_SMD:C_0201_0603Metric
- C24: renamed from C23; footprint (none) -> Capacitor_SMD:C_0201_0603Metric
- C25: renamed from C24; footprint (none) -> Capacitor_SMD:C_0201_0603Metric
- C26: renamed from C25; footprint (none) -> Capacitor_SMD:C_0201_0603Metric
- C27: renamed from C26; footprint (none) -> Capacitor_SMD:C_0201_0603Metric
- C28: renamed from C27; footprint (none) -> Capacitor_SMD:C_0201_0603Metric
- C29: renamed from C28; footprint (none) -> Capacitor_SMD:C_0201_0603Metric
- R10, R11, R12, R13, R14, R15, R16, R5, R8, R9: footprint (none) -> Resistor_SMD:R_0201_0603Metric
- R17: footprint (none) -> Resistor_SMD:R_0201_0603Metric_Pad0.64x0.40mm_HandSolder
- R6: renamed from R7; footprint (none) -> Resistor_SMD:R_0201_0603Metric
- R7: renamed from R6; footprint (none) -> Resistor_SMD:R_0201_0603Metric
- renumbered S2 to S1, S3 to S2
Connections:
- net +3V3: now also C30.2, C32.1, J4.12, J5.5 (Pin_5), R18.1, S10.1 (COM_1), S11.1 (COM_1), S12.1 (COM_1), S13.1 (COM_1), S3.1 (COM_1), S4.1 (COM_1), S5.1 (COM_1), S6.1 (COM_1), S7.1 (COM_1), S8.1 (COM_1), S9.1 (COM_1)
- net BTN.A: now also S3.3 (NO_1)
- net BTN.B: now also S4.3 (NO_1)
- net BTN.L1: now also S12.3 (NO_1)
- net BTN.PS: now also S11.3 (NO_1)
- net BTN.R1: now also S13.3 (NO_1)
- net BTN.X: now also S5.3 (NO_1)
- net BTN.Y: now also S6.3 (NO_1)
- net DPAD.E: now also S10.3 (NO_1)
- net DPAD.N: now also S7.3 (NO_1)
- net DPAD.S: now also S8.3 (NO_1)
- net DPAD.W: now also S9.3 (NO_1)
- net GND: now also C30.1, J4.11, J5.4 (Pin_4)
- new net: C32.2, J5.6 (Pin_6)
- new net: J5.1 (Pin_1), R18.2
- new net: C31.1, J5.7 (Pin_7)
- new net: C31.2, J5.8 (Pin_8)
- new net LCD.SCL: J5.2 (Pin_2)
- new net LCD.SDA: J5.3 (Pin_3)
- new net TPad.BTN1: J4.8
- new net TPad.BTN2: J4.6
- new net TPad.BTN3: J4.7
- new net TPad.DR: J4.4
- new net TPad.MISO: J4.2
- new net TPad.MOSI: J4.5
- new net TPad.SCK: J4.1
- new net TPad.SS: J4.3
- no-connect marks 12 -> 37
Other:
- note added: "AQM1602A"
- note added: "CAP1N"
- note added: "CAP1P"
- note added: "LCD"
- note added: "RESET"
- note added: "SCL"
- note added: "SDA"
- note added: "TM035035 TrackPad"
- note added: "V0"
- note added: "VDD"
- note added: "VOUT"
- note added: "VSS"
- title: (none) -> STM32マイコンゲームコントローラ
- moved on the sheet: C20, C21, C22, R10, R8, R9

Commit message: Schematics Done
Parts:
- added C33, C34: 100n, Capacitor_SMD:C_0201_0603Metric, symbol Device:C_Small
- added LED1, LED2: IN-S66TBTRGB, RGB_LED:INS66TBTRGB, symbol IN-S66TBTRGB:IN-S66TBTRGB
- added R19, R22: 470, Resistor_SMD:R_0201_0603Metric, symbol Device:R_Small
- added R20, R23: 270, Resistor_SMD:R_0201_0603Metric, symbol Device:R_Small
- added R21, R4: 330, Resistor_SMD:R_0201_0603Metric, symbol Device:R_Small
Connections:
- net +3V3: now also C33.1, C34.1, LED1.1 (COM+), LED2.1 (COM+)
- net GND: now also C33.2, C34.2
- new net: LED1.2 (K_RED), R20.1
- new net: LED1.3 (K_BLUE), R4.1
- new net: LED1.4 (K_GREEN), R19.1
- new net: LED2.4 (K_GREEN), R22.1
- new net: LED2.2 (K_RED), R23.1
- new net: LED2.3 (K_BLUE), R21.1
- new net RGB_A.Blue: R4.2
- new net RGB_A.Green: R19.2
- new net RGB_A.Red: R20.2
- new net RGB_B.Blue: R21.2
- new net RGB_B.Green: R22.2
- new net RGB_B.Red: R23.2
Other:
- note added: "RGB LEDs"
- moved on the sheet: C30, C31, C32, J4, J5, R18
